Commit message: Correct URDF for pneumatic end effector

File: examples/robots/iiwa7_description.urdf.xacro (robot description, xacro)
@@ -261,5 +261,5 @@
             <parent link="${robot_name}_link_7"/>
             <child link="${robot_name}_link_ee"/>
-            <origin xyz="0 0 0.035" rpy="0 0 0"/>
+            <origin xyz="0 0 0.07" rpy="0 0 0"/>
         </joint>
         <link name="${robot_name}_link_ee">
